File: hardware/ESP-12E.sch (KiCad schematic (older format))
At the start: 13 parts, among them SW1 SW_RESET,2_leg,SMD, SW2 SW_RESET,2_leg,SMD, U2 ESP-12E

Commit message: update,
Parts:
- added J?: TTL_HEADER, footprint-lib:TTL_HEADER, symbol taobao-components:TTL_HEADER
Connections:
- net GND: now also J?.GND
- net RXD: now also J?.RX
- net TXD: now also J?.TX
Changed lines of the file:
@@
 $Descr A4 11693 8268
 encoding utf-8
-Sheet 7 10
+Sheet 7 9
 Title ""
 Date ""
@@
 Wire Wire Line
 	2650 1350 3200 1350
-$Sheet
-S 9250 5400 900  700
-U 5CF690E7
-F0 "CP2102" 50
-F1 "CP2102.sch" 50
-F2 "RESET" I L 9250 5550 50
-F3 "GPIO0" I L 9250 5650 50
-F4 "RXD" I L 9250 5850 50
-F5 "TXD" I L 9250 5950 50
-$EndSheet
 Text Label 8850 5950 0    50   ~ 0
 TXD
@@
 Wire Wire Line
 	9250 5850 8850 5850
-Text Label 8850 5650 0    50   ~ 0
-GPIO0
-Wire Wire Line
-	8850 5650 9250 5650
-Text Label 8850 5550 0    50   ~ 0
-RESET
-Wire Wire Line
-	8850 5550 9250 5550
 Text HLabel 2650 1550 0    50   Input ~ 0
 CS
@@
 Text HLabel 2650 2600 0    50   Input ~ 0
 IO5
+$Comp
+L taobao-components:TTL_HEADER J?
+U 1 1 5CF7E930
+P 9250 5950
+F 0 "J?" H 9022 5882 50  0000 R CNN
+F 1 "TTL_HEADER" H 9022 5973 50  0000 R CNN
+F 2 "footprint-lib:TTL_HEADER" H 9250 5550 50  0001 C CNN
+F 3 "" H 9050 5950 50  0001 C CNN
+	1    9250 5950
+	-1   0    0    1
+$EndComp
+$Comp
+L power:GND #PWR?
+U 1 1 5CF7F9B3
+P 9150 6250
+F 0 "#PWR?" H 9150 6000 50  0001 C CNN
+F 1 "GND" H 9155 6077 50  0000 C CNN
+F 2 "" H 9150 6250 50  0001 C CNN
+F 3 "" H 9150 6250 50  0001 C CNN
+	1    9150 6250
+	1    0    0    -1
+$EndComp
+Wire Wire Line
+	9150 6250 9150 6050
+Wire Wire Line
+	9150 6050 9250 6050
 $EndSCHEMATC

Commit message: update,
Parts:
- removed R16: R561, symbol taobao-r:R561
- added R13: R561,0603, Resistor_SMD:R_0603_1608Metric_Pad1.05x0.95mm_HandSolder, symbol taobao-r:R561,0603
- gave numbers to parts that had none: 1
- renumbered R12 to R10, R14 to R11, R15 to R12, R9 to R7, R10 to R8, R11 to R9
Connections:
- net +3V3: now also R13.1
- net at D4.2 (A): now also R13.2
Changed lines of the file:
@@
 $EndComp
 $Comp
-L power:+3V3 #PWR0128
+L power:+3V3 #PWR026
 U 1 1 5CFAE4AE
 P 6150 2300
-F 0 "#PWR0128" H 6150 2150 50  0001 C CNN
+F 0 "#PWR026" H 6150 2150 50  0001 C CNN
 F 1 "+3V3" H 6165 2473 50  0000 C CNN
 F 2 "" H 6150 2300 50  0001 C CNN
@@
 $EndComp
 $Comp
-L power:GND #PWR0129
+L power:GND #PWR030
 U 1 1 5CFAE821
 P 6150 4550
-F 0 "#PWR0129" H 6150 4300 50  0001 C CNN
+F 0 "#PWR030" H 6150 4300 50  0001 C CNN
 F 1 "GND" H 6155 4377 50  0000 C CNN
 F 2 "" H 6150 4550 50  0001 C CNN
@@
 	6150 2300 6150 2450
 $Comp
-L power:+3V3 #PWR0130
+L power:+3V3 #PWR023
 U 1 1 5CFAEF78
 P 5900 1950
-F 0 "#PWR0130" H 5900 1800 50  0001 C CNN
+F 0 "#PWR023" H 5900 1800 50  0001 C CNN
 F 1 "+3V3" V 5915 2078 50  0000 L CNN
 F 2 "" H 5900 1950 50  0001 C CNN
@@
 $EndComp
 $Comp
-L power:GND #PWR0131
+L power:GND #PWR024
 U 1 1 5CFAF616
 P 6500 1950
-F 0 "#PWR0131" H 6500 1700 50  0001 C CNN
+F 0 "#PWR024" H 6500 1700 50  0001 C CNN
 F 1 "GND" V 6505 1822 50  0000 R CNN
 F 2 "" H 6500 1950 50  0001 C CNN
@@
 	4050 3100 4800 3100
 $Comp
-L power:+3V3 #PWR0132
+L power:+3V3 #PWR031
 U 1 1 5CFB5123
 P 800 5250
-F 0 "#PWR0132" H 800 5100 50  0001 C CNN
+F 0 "#PWR031" H 800 5100 50  0001 C CNN
 F 1 "+3V3" H 815 5423 50  0000 C CNN
 F 2 "" H 800 5250 50  0001 C CNN
 F 3 "" H 800 5250 50  0001 C CNN
 	1    800  5250
-	1    0    0    -1
-$EndComp
-$Comp
-L taobao-r:R561 R16
-U 1 1 5CFB53F7
-P 800 5500
-F 0 "R16" H 859 5546 50  0000 L CNN
-F 1 "R561" H 859 5455 50  0000 L CNN
-F 2 "" H 800 5500 50  0001 C CNN
-F 3 "~" H 800 5500 50  0001 C CNN
-	1    800  5500
 	1    0    0    -1
 $EndComp
@@
 	800  5400 800  5250
 $Comp
-L taobao-r:R102,0603 R12
+L taobao-r:R102,0603 R10
 U 1 1 5CFB90C1
 P 8100 3300
-F 0 "R12" V 8150 3450 50  0000 C CNN
+F 0 "R10" V 8150 3450 50  0000 C CNN
 F 1 "R102,0603" V 8200 3700 50  0000 C CNN
 F 2 "Resistor_SMD:R_0603_1608Metric_Pad1.05x0.95mm_HandSolder" H 8100 3300 50  0001 C CNN
@@
 $EndComp
 $Comp
-L power:+3V3 #PWR0134
+L power:+3V3 #PWR028
 U 1 1 5CFB93DB
 P 8700 3050
-F 0 "#PWR0134" H 8700 2900 50  0001 C CNN
+F 0 "#PWR028" H 8700 2900 50  0001 C CNN
 F 1 "+3V3" H 8715 3223 50  0000 C CNN
 F 2 "" H 8700 3050 50  0001 C CNN
@@
 RESET
 $Comp
-L taobao-r:R471,0603 R14
+L taobao-r:R471,0603 R11
 U 1 1 5CFC1D26
 P 2300 3550
-F 0 "R14" H 2359 3596 50  0000 L CNN
+F 0 "R11" H 2359 3596 50  0000 L CNN
 F 1 "R471,0603" H 2359 3505 50  0000 L CNN
 F 2 "Resistor_SMD:R_0603_1608Metric_Pad1.05x0.95mm_HandSolder" H 2300 3550 50  0001 C CNN
@@
 $EndComp
 $Comp
-L power:GND #PWR0135
+L power:GND #PWR029
 U 1 1 5CFC292C
 P 2000 4300
-F 0 "#PWR0135" H 2000 4050 50  0001 C CNN
+F 0 "#PWR029" H 2000 4050 50  0001 C CNN
 F 1 "GND" H 2005 4127 50  0000 C CNN
 F 2 "" H 2000 4300 50  0001 C CNN
@@
 	2300 3350 2300 3450
 $Comp
-L power:+3V3 #PWR0136
+L power:+3V3 #PWR025
 U 1 1 5CFC79FD
 P 1750 2100
-F 0 "#PWR0136" H 1750 1950 50  0001 C CNN
+F 0 "#PWR025" H 1750 1950 50  0001 C CNN
 F 1 "+3V3" H 1765 2273 50  0000 C CNN
 F 2 "" H 1750 2100 50  0001 C CNN
@@
 $EndComp
 $Comp
-L taobao-r:R471,0603 R9
+L taobao-r:R471,0603 R7
 U 1 1 5CFC87CD
 P 1750 2350
-F 0 "R9" H 1809 2396 50  0000 L CNN
+F 0 "R7" H 1809 2396 50  0000 L CNN
 F 1 "R471,0603" H 1809 2305 50  0000 L CNN
 F 2 "Resistor_SMD:R_0603_1608Metric_Pad1.05x0.95mm_HandSolder" H 1750 2350 50  0001 C CNN
@@
 $EndComp
 $Comp
-L taobao-r:R0,0603 R11
+L taobao-r:R0,0603 R9
 U 1 1 5CFC9CB3
 P 1750 3050
-F 0 "R11" H 1809 3096 50  0000 L CNN
+F 0 "R9" H 1809 3096 50  0000 L CNN
 F 1 "R0,0603" H 1809 3005 50  0000 L CNN
 F 2 "Resistor_SMD:R_0603_1608Metric_Pad1.05x0.95mm_HandSolder" H 1750 3050 50  0001 C CNN
@@
 GPIO0
 $Comp
-L taobao-r:R471,0603 R15
+L taobao-r:R471,0603 R12
 U 1 1 5CFE09F2
 P 1900 5300
-F 0 "R15" H 1959 5346 50  0000 L CNN
+F 0 "R12" H 1959 5346 50  0000 L CNN
 F 1 "R471,0603" H 1959 5255 50  0000 L CNN
 F 2 "Resistor_SMD:R_0603_1608Metric_Pad1.05x0.95mm_HandSolder" H 1900 5300 50  0001 C CNN
@@
 $EndComp
 $Comp
-L power:GND #PWR0137
+L power:GND #PWR032
 U 1 1 5CFE144C
 P 1900 6050
-F 0 "#PWR0137" H 1900 5800 50  0001 C CNN
+F 0 "#PWR032" H 1900 5800 50  0001 C CNN
 F 1 "GND" H 1905 5877 50  0000 C CNN
 F 2 "" H 1900 6050 50  0001 C CNN
@@
 	1900 5100 1900 5200
 $Comp
-L power:+3V3 #PWR0138
+L power:+3V3 #PWR027
 U 1 1 5CFE883F
 P 3750 2550
-F 0 "#PWR0138" H 3750 2400 50  0001 C CNN
+F 0 "#PWR027" H 3750 2400 50  0001 C CNN
 F 1 "+3V3" H 3765 2723 50  0000 C CNN
 F 2 "" H 3750 2550 50  0001 C CNN
@@
 $EndComp
 $Comp
-L taobao-r:R102,0603 R10
+L taobao-r:R102,0603 R8
 U 1 1 5CFE8BA8
 P 3750 2800
-F 0 "R10" H 3692 2846 50  0000 R CNN
+F 0 "R8" H 3692 2846 50  0000 R CNN
 F 1 "R102,0603" H 3692 2755 50  0000 R CNN
 F 2 "Resistor_SMD:R_0603_1608Metric_Pad1.05x0.95mm_HandSolder" H 3750 2800 50  0001 C CNN
@@
 IO5
 $Comp
-L taobao-components:TTL_HEADER J?
+L taobao-components:TTL_HEADER J5
 U 1 1 5CF7E930
 P 9250 5950
-F 0 "J?" H 9022 5882 50  0000 R CNN
+F 0 "J5" H 9022 5882 50  0000 R CNN
 F 1 "TTL_HEADER" H 9022 5973 50  0000 R CNN
 F 2 "footprint-lib:TTL_HEADER" H 9250 5550 50  0001 C CNN
@@
 $EndComp
 $Comp
-L power:GND #PWR?
+L power:GND #PWR033
 U 1 1 5CF7F9B3
 P 9150 6250
-F 0 "#PWR?" H 9150 6000 50  0001 C CNN
+F 0 "#PWR033" H 9150 6000 50  0001 C CNN
 F 1 "GND" H 9155 6077 50  0000 C CNN
 F 2 "" H 9150 6250 50  0001 C CNN
@@
 Wire Wire Line
 	9150 6050 9250 6050
+$Comp
+L taobao-r:R561,0603 R13
+U 1 1 5CF85C5A
+P 800 5500
+F 0 "R13" H 859 5546 50  0000 L CNN
+F 1 "R561,0603" H 859 5455 50  0000 L CNN
+F 2 "Resistor_SMD:R_0603_1608Metric_Pad1.05x0.95mm_HandSolder" H 800 5500 50  0001 C CNN
+F 3 "~" H 800 5500 50  0001 C CNN
+	1    800  5500
+	1    0    0    -1
+$EndComp
 $EndSCHEMATC
