File: hardware/gpio.sch (KiCad schematic (older format))
At the start: 1 part, among them J6 IO

Commit message: update,
Parts:
- J7: renamed from J6; footprint (none) -> Connector_PinHeader_2.54mm:PinHeader_1x07_P2.54mm_Vertical
Changed lines of the file:
@@
 $EndDescr
 $Comp
-L Connector:Conn_01x07_Female J6
+L Connector:Conn_01x07_Female J7
 U 1 1 5CF9E2C4
 P 3200 2000
-F 0 "J6" H 3228 1976 50  0000 L CNN
+F 0 "J7" H 3228 1976 50  0000 L CNN
 F 1 "IO" H 3228 1885 50  0000 L CNN
-F 2 "" H 3200 2000 50  0001 C CNN
+F 2 "Connector_PinHeader_2.54mm:PinHeader_1x07_P2.54mm_Vertical" H 3200 2000 50  0001 C CNN
 F 3 "~" H 3200 2000 50  0001 C CNN
 	1    3200 2000
@@
 $EndComp
 $Comp
-L power:+5V #PWR0126
+L power:+5V #PWR048
 U 1 1 5CF9E63D
 P 2700 2400
-F 0 "#PWR0126" H 2700 2250 50  0001 C CNN
+F 0 "#PWR048" H 2700 2250 50  0001 C CNN
 F 1 "+5V" H 2715 2573 50  0000 C CNN
 F 2 "" H 2700 2400 50  0001 C CNN
@@
 $EndComp
 $Comp
-L power:GND #PWR0127
+L power:GND #PWR047
 U 1 1 5CF9EAF1
 P 2700 1600
-F 0 "#PWR0127" H 2700 1350 50  0001 C CNN
+F 0 "#PWR047" H 2700 1350 50  0001 C CNN
 F 1 "GND" H 2705 1427 50  0000 C CNN
 F 2 "" H 2700 1600 50  0001 C CNN
