File: hardware/i2c.sch (KiCad schematic (older format))
At the start: 2 parts, among them J2 I2C

Commit message: update,
Parts:
- J2: footprint (none) -> Connector_PinHeader_2.54mm:PinHeader_1x04_P2.54mm_Vertical
Changed lines of the file:
@@
 F 0 "J2" H 2392 2735 50  0000 C CNN
 F 1 "I2C" H 2392 2644 50  0000 C CNN
-F 2 "" H 2500 2450 50  0001 C CNN
+F 2 "Connector_PinHeader_2.54mm:PinHeader_1x04_P2.54mm_Vertical" H 2500 2450 50  0001 C CNN
 F 3 "~" H 2500 2450 50  0001 C CNN
 	1    2500 2450
@@
 SCL
 $Comp
-L power:GND #PWR0113
+L power:GND #PWR014
 U 1 1 5CF906FC
 P 3100 2250
-F 0 "#PWR0113" H 3100 2000 50  0001 C CNN
+F 0 "#PWR014" H 3100 2000 50  0001 C CNN
 F 1 "GND" H 3105 2077 50  0000 C CNN
 F 2 "" H 3100 2250 50  0001 C CNN
@@
 	1050 1100 1500 1100
 $Comp
-L power:+3V3 #PWR0114
+L power:+3V3 #PWR013
 U 1 1 5CF91D29
 P 3450 1650
-F 0 "#PWR0114" H 3450 1500 50  0001 C CNN
+F 0 "#PWR013" H 3450 1500 50  0001 C CNN
 F 1 "+3V3" H 3465 1823 50  0000 C CNN
 F 2 "" H 3450 1650 50  0001 C CNN
@@
 	3500 2200 3500 2550
 $Comp
-L power:+5V #PWR0115
+L power:+5V #PWR015
 U 1 1 5CFA5633
 P 3100 2800
-F 0 "#PWR0115" H 3100 2650 50  0001 C CNN
+F 0 "#PWR015" H 3100 2650 50  0001 C CNN
 F 1 "+5V" H 3115 2973 50  0000 C CNN
 F 2 "" H 3100 2800 50  0001 C CNN
