File: hardware/SDCARD.sch (KiCad schematic (older format))
At the start: 7 parts

Commit message: update,
Parts:
- J6: renamed from J?; footprint (none) -> Connector_PinHeader_2.54mm:PinHeader_1x08_P2.54mm_Vertical
- gave numbers to parts that had none: 6
Changed lines of the file:
@@
 $EndDescr
 $Comp
-L taobao-components:TF_CARD_SOCKET,SELF_EJECT U?
+L taobao-components:TF_CARD_SOCKET,SELF_EJECT U4
 U 1 1 5CFD75CD
 P 5950 2350
-F 0 "U?" H 6678 2396 50  0000 L CNN
+F 0 "U4" H 6678 2396 50  0000 L CNN
 F 1 "TF_CARD_SOCKET,SELF_EJECT" H 6678 2305 50  0000 L CNN
 F 2 "footprint-lib:SUNTECH_ST-TF-003A" H 6050 2450 50  0001 C CNN
@@
 $EndComp
 $Comp
-L power:GND #PWR?
+L power:GND #PWR043
 U 1 1 5CFD7960
 P 5550 2950
-F 0 "#PWR?" H 5550 2700 50  0001 C CNN
+F 0 "#PWR043" H 5550 2700 50  0001 C CNN
 F 1 "GND" H 5555 2777 50  0000 C CNN
 F 2 "" H 5550 2950 50  0001 C CNN
@@
 Connection ~ 5550 2800
 $Comp
-L power:+3V3 #PWR?
+L power:+3V3 #PWR038
 U 1 1 5CFD813E
 P 5500 1750
-F 0 "#PWR?" H 5500 1600 50  0001 C CNN
+F 0 "#PWR038" H 5500 1600 50  0001 C CNN
 F 1 "+3V3" H 5515 1923 50  0000 C CNN
 F 2 "" H 5500 1750 50  0001 C CNN
@@
 	5750 2700 5150 2700
 $Comp
-L power:+3V3 #PWR?
+L power:+3V3 #PWR036
 U 1 1 5CFF5AB6
 P 6050 1600
-F 0 "#PWR?" H 6050 1450 50  0001 C CNN
+F 0 "#PWR036" H 6050 1450 50  0001 C CNN
 F 1 "+3V3" V 6065 1728 50  0000 L CNN
 F 2 "" H 6050 1600 50  0001 C CNN
@@
 $EndComp
 $Comp
-L power:GND #PWR?
+L power:GND #PWR037
 U 1 1 5CFF622C
 P 6550 1600
-F 0 "#PWR?" H 6550 1350 50  0001 C CNN
+F 0 "#PWR037" H 6550 1350 50  0001 C CNN
 F 1 "GND" V 6555 1472 50  0000 R CNN
 F 2 "" H 6550 1600 50  0001 C CNN
@@
 $EndComp
 $Comp
-L taobao-cp:CP1uf,50V C?
+L taobao-cp:CP1uf,50V C7
 U 1 1 5CFF6905
 P 6300 1600
-F 0 "C?" V 6525 1600 50  0000 C CNN
+F 0 "C7" V 6525 1600 50  0000 C CNN
 F 1 "CP1uf,50V" V 6434 1600 50  0000 C CNN
 F 2 "Capacitor_SMD:CP_Elec_4x5.3" H 6300 1600 50  0001 C CNN
@@
 	1600 4100 2300 4100
 $Comp
-L power:GND #PWR?
+L power:GND #PWR046
 U 1 1 5CFFC8B7
 P 1600 3950
-F 0 "#PWR?" H 1600 3700 50  0001 C CNN
+F 0 "#PWR046" H 1600 3700 50  0001 C CNN
 F 1 "GND" H 1605 3777 50  0000 C CNN
 F 2 "" H 1600 3950 50  0001 C CNN
@@
 	1800 4000 2300 4000
 $Comp
-L power:+3V3 #PWR?
+L power:+3V3 #PWR045
 U 1 1 5CFFB34E
 P 1800 3900
-F 0 "#PWR?" H 1800 3750 50  0001 C CNN
+F 0 "#PWR045" H 1800 3750 50  0001 C CNN
 F 1 "+3V3" H 1815 4073 50  0000 C CNN
 F 2 "" H 1800 3900 50  0001 C CNN
@@
 	1950 3750 1950 3900
 $Comp
-L power:GND #PWR?
+L power:GND #PWR044
 U 1 1 5CFFA7A7
 P 1950 3750
-F 0 "#PWR?" H 1950 3500 50  0001 C CNN
+F 0 "#PWR044" H 1950 3500 50  0001 C CNN
 F 1 "GND" H 1955 3577 50  0000 C CNN
 F 2 "" H 1950 3750 50  0001 C CNN
@@
 $EndComp
 $Comp
-L Connector:Conn_01x08_Female J?
+L Connector:Conn_01x08_Female J6
 U 1 1 5CFF8EDD
 P 2500 4200
-F 0 "J?" H 2528 4176 50  0000 L CNN
+F 0 "J6" H 2528 4176 50  0000 L CNN
 F 1 "TF_HEADER" H 2528 4085 50  0000 L CNN
-F 2 "" H 2500 4200 50  0001 C CNN
+F 2 "Connector_PinHeader_2.54mm:PinHeader_1x08_P2.54mm_Vertical" H 2500 4200 50  0001 C CNN
 F 3 "~" H 2500 4200 50  0001 C CNN
 	1    2500 4200
@@
 	2650 1450 2750 1450
 $Comp
-L taobao-c:C106,0603 C?
+L taobao-c:C106,0603 C6
 U 1 1 5CFF1866
 P 2850 1450
-F 0 "C?" V 2621 1450 50  0000 C CNN
+F 0 "C6" V 2621 1450 50  0000 C CNN
 F 1 "C106,0603" V 2712 1450 50  0000 C CNN
 F 2 "Capacitor_SMD:C_0603_1608Metric_Pad1.05x0.95mm_HandSolder" H 2850 1450 50  0001 C CNN
@@
 $EndComp
 $Comp
-L power:GND #PWR?
+L power:GND #PWR035
 U 1 1 5CFF1367
 P 3050 1450
-F 0 "#PWR?" H 3050 1200 50  0001 C CNN
+F 0 "#PWR035" H 3050 1200 50  0001 C CNN
 F 1 "GND" V 3055 1322 50  0000 R CNN
 F 2 "" H 3050 1450 50  0001 C CNN
@@
 $EndComp
 $Comp
-L power:+3V3 #PWR?
+L power:+3V3 #PWR034
 U 1 1 5CFF0AAE
 P 2650 1450
-F 0 "#PWR?" H 2650 1300 50  0001 C CNN
+F 0 "#PWR034" H 2650 1300 50  0001 C CNN
 F 1 "+3V3" V 2665 1578 50  0000 L CNN
 F 2 "" H 2650 1450 50  0001 C CNN
@@
 	3550 2550 3850 2550
 $Comp
-L taobao-led:LED_GREEN,0603 D?
+L taobao-led:LED_GREEN,0603 D5
 U 1 1 5CFEA629
 P 4200 2550
-F 0 "D?" H 4200 2345 50  0000 C CNN
+F 0 "D5" H 4200 2345 50  0000 C CNN
 F 1 "LED_GREEN,0603" H 4200 2436 50  0000 C CNN
 F 2 "footprint-lib:LED_0603_1608Metric" V 4200 2550 50  0001 C CNN
@@
 $EndComp
 $Comp
-L taobao-r:R102,0603 R?
+L taobao-r:R102,0603 R14
 U 1 1 5CFE9EC7
 P 3950 2550
-F 0 "R?" V 3754 2550 50  0000 C CNN
+F 0 "R14" V 3754 2550 50  0000 C CNN
 F 1 "R102,0603" V 3845 2550 50  0000 C CNN
 F 2 "Resistor_SMD:R_0603_1608Metric_Pad1.05x0.95mm_HandSolder" H 3950 2550 50  0001 C CNN
@@
 	3750 2150 3550 2150
 $Comp
-L power:GND #PWR?
+L power:GND #PWR040
 U 1 1 5CFDCCF6
 P 3750 2150
-F 0 "#PWR?" H 3750 1900 50  0001 C CNN
+F 0 "#PWR040" H 3750 1900 50  0001 C CNN
 F 1 "GND" V 3755 2022 50  0000 R CNN
 F 2 "" H 3750 2150 50  0001 C CNN
@@
 	3750 2450 3550 2450
 $Comp
-L power:GND #PWR?
+L power:GND #PWR041
 U 1 1 5CFDC349
 P 3750 2450
-F 0 "#PWR?" H 3750 2200 50  0001 C CNN
+F 0 "#PWR041" H 3750 2200 50  0001 C CNN
 F 1 "GND" V 3755 2322 50  0000 R CNN
 F 2 "" H 3750 2450 50  0001 C CNN
@@
 	1900 1800 1900 1950
 $Comp
-L power:+3V3 #PWR?
+L power:+3V3 #PWR039
 U 1 1 5CFD991A
 P 1900 1800
-F 0 "#PWR?" H 1900 1650 50  0001 C CNN
+F 0 "#PWR039" H 1900 1650 50  0001 C CNN
 F 1 "+3V3" H 1915 1973 50  0000 C CNN
 F 2 "" H 1900 1800 50  0001 C CNN
@@
 	2150 2650 1950 2650
 $Comp
-L power:GND #PWR?
+L power:GND #PWR042
 U 1 1 5CFD92D6
 P 1950 2850
-F 0 "#PWR?" H 1950 2600 50  0001 C CNN
+F 0 "#PWR042" H 1950 2600 50  0001 C CNN
 F 1 "GND" H 1955 2677 50  0000 C CNN
 F 2 "" H 1950 2850 50  0001 C CNN
@@
 DI
 $Comp
-L taobao-components:CD74HC4050 U?
+L taobao-components:CD74HC4050 U3
 U 1 1 5CFD5C32
 P 2850 2300
-F 0 "U?" H 2850 3015 50  0000 C CNN
+F 0 "U3" H 2850 3015 50  0000 C CNN
 F 1 "CD74HC4050" H 2850 2924 50  0000 C CNN
 F 2 "" H 2850 2300 50  0001 C CNN

Commit message: update,
Parts:
- U3: footprint (none) -> footprint-lib:74HCT4050_SOP16
Changed lines of the file:
@@
 U 1 1 5CFEA629
 P 4200 2550
-F 0 "D5" H 4200 2345 50  0000 C CNN
-F 1 "LED_GREEN,0603" H 4200 2436 50  0000 C CNN
+F 0 "D5" H 4200 2693 50  0000 C CNN
+F 1 "LED_GREEN,0603" H 4200 2784 50  0000 C CNN
 F 2 "footprint-lib:LED_0603_1608Metric" V 4200 2550 50  0001 C CNN
 F 3 "" V 4200 2550 50  0001 C CNN
@@
 P 3750 2450
 F 0 "#PWR041" H 3750 2200 50  0001 C CNN
-F 1 "GND" V 3755 2322 50  0000 R CNN
+F 1 "GND" V 3883 2413 50  0000 C CNN
 F 2 "" H 3750 2450 50  0001 C CNN
 F 3 "" H 3750 2450 50  0001 C CNN
@@
 Text Label 1700 2350 0    50   ~ 0
 DI
-$Comp
-L taobao-components:CD74HC4050 U3
-U 1 1 5CFD5C32
-P 2850 2300
-F 0 "U3" H 2850 3015 50  0000 C CNN
-F 1 "CD74HC4050" H 2850 2924 50  0000 C CNN
-F 2 "" H 2850 2300 50  0001 C CNN
-F 3 "" H 2850 2300 50  0001 C CNN
-	1    2850 2300
-	1    0    0    -1
-$EndComp
 Wire Wire Line
 	1600 1000 1150 1000
@@
 EndData
 $EndBitmap
+$Comp
+L taobao-components:CD74HC4050 U3
+U 1 1 5CF97526
+P 2850 2300
+F 0 "U3" H 2850 3015 50  0000 C CNN
+F 1 "CD74HC4050" H 2850 2924 50  0000 C CNN
+F 2 "footprint-lib:74HCT4050_SOP16" H 2850 1500 50  0001 C CNN
+F 3 "" H 2850 2300 50  0001 C CNN
+	1    2850 2300
+	1    0    0    -1
+$EndComp
 $EndSCHEMATC
