File: hardware/analog.sch (KiCad schematic (older format))
At the start: 3 parts, among them J3 ADC

Commit message: update,
Parts:
- J3: footprint (none) -> Connector_PinHeader_2.54mm:PinHeader_1x03_P2.54mm_Vertical
Changed lines of the file:
@@
 F 0 "J3" H 2392 2585 50  0000 C CNN
 F 1 "ADC" H 2392 2494 50  0000 C CNN
-F 2 "" H 2500 2300 50  0001 C CNN
+F 2 "Connector_PinHeader_2.54mm:PinHeader_1x03_P2.54mm_Vertical" H 2500 2300 50  0001 C CNN
 F 3 "~" H 2500 2300 50  0001 C CNN
 	1    2500 2300
@@
 $EndComp
 $Comp
-L power:GND #PWR0116
+L power:GND #PWR016
 U 1 1 5CF93EF7
 P 3000 2000
-F 0 "#PWR0116" H 3000 1750 50  0001 C CNN
+F 0 "#PWR016" H 3000 1750 50  0001 C CNN
 F 1 "GND" H 3005 1827 50  0000 C CNN
 F 2 "" H 3000 2000 50  0001 C CNN
@@
 $EndComp
 $Comp
-L power:+3V3 #PWR0117
+L power:+3V3 #PWR017
 U 1 1 5CF94172
 P 3000 2650
-F 0 "#PWR0117" H 3000 2500 50  0001 C CNN
+F 0 "#PWR017" H 3000 2500 50  0001 C CNN
 F 1 "+3V3" H 3015 2823 50  0000 C CNN
 F 2 "" H 3000 2650 50  0001 C CNN
@@
 	3650 2300 4200 2300
 $Comp
-L power:GND #PWR0118
+L power:GND #PWR018
 U 1 1 5CF954CA
 P 3650 2700
-F 0 "#PWR0118" H 3650 2450 50  0001 C CNN
+F 0 "#PWR018" H 3650 2450 50  0001 C CNN
 F 1 "GND" H 3655 2527 50  0000 C CNN
 F 2 "" H 3650 2700 50  0001 C CNN
