File: hardware/one-wire.sch (KiCad schematic (older format))
At the start: 3 parts, among them J4 ONE_WIRE

Commit message: update,
Parts:
- J4: footprint (none) -> Connector_PinHeader_2.54mm:PinHeader_1x03_P2.54mm_Vertical
Changed lines of the file:
@@
 F 0 "J4" H 3228 1876 50  0000 L CNN
 F 1 "ONE_WIRE" H 3228 1785 50  0000 L CNN
-F 2 "" H 3200 1850 50  0001 C CNN
+F 2 "Connector_PinHeader_2.54mm:PinHeader_1x03_P2.54mm_Vertical" H 3200 1850 50  0001 C CNN
 F 3 "~" H 3200 1850 50  0001 C CNN
 	1    3200 1850
@@
 $EndComp
 $Comp
-L power:GND #PWR0119
+L power:GND #PWR021
 U 1 1 5CF962C9
 P 2600 1550
-F 0 "#PWR0119" H 2600 1300 50  0001 C CNN
+F 0 "#PWR021" H 2600 1300 50  0001 C CNN
 F 1 "GND" H 2605 1377 50  0000 C CNN
 F 2 "" H 2600 1550 50  0001 C CNN
@@
 $EndComp
 $Comp
-L power:+3V3 #PWR0120
+L power:+3V3 #PWR022
 U 1 1 5CF96695
 P 2600 2450
-F 0 "#PWR0120" H 2600 2300 50  0001 C CNN
+F 0 "#PWR022" H 2600 2300 50  0001 C CNN
 F 1 "+3V3" H 2615 2623 50  0000 C CNN
 F 2 "" H 2600 2450 50  0001 C CNN
@@
 	900  900  1450 900
 $Comp
-L power:+3V3 #PWR0121
+L power:+3V3 #PWR019
 U 1 1 5CF993E4
 P 2200 1200
-F 0 "#PWR0121" H 2200 1050 50  0001 C CNN
+F 0 "#PWR019" H 2200 1050 50  0001 C CNN
 F 1 "+3V3" V 2215 1328 50  0000 L CNN
 F 2 "" H 2200 1200 50  0001 C CNN
@@
 $EndComp
 $Comp
-L power:GND #PWR0122
+L power:GND #PWR020
 U 1 1 5CF9965F
 P 2650 1200
-F 0 "#PWR0122" H 2650 950 50  0001 C CNN
+F 0 "#PWR020" H 2650 950 50  0001 C CNN
 F 1 "GND" V 2655 1072 50  0000 R CNN
 F 2 "" H 2650 1200 50  0001 C CNN
