File: hardware/power.sch (KiCad schematic (older format))
At the start: 13 parts, among them J1 Vin, U1 AMS1117-3.3

Commit message: update,
Parts:
- removed JP1: 5V_EN, symbol Device:Jumper_NO_Small
- removed JP2: 3V3_EN, symbol Device:Jumper_NO_Small
- added JP1: 5V_EN, Jumper:SolderJumper-2_P1.3mm_Open_RoundedPad1.0x1.5mm, symbol my_solder_jumper:SolderJumper_2_Open_round
- added JP2: 3V3_EN, Jumper:SolderJumper-2_P1.3mm_Open_RoundedPad1.0x1.5mm, symbol my_solder_jumper:SolderJumper_2_Open_round
- J1: footprint (none) -> Connector_PinHeader_2.54mm:PinHeader_1x02_P2.54mm_Vertical
Connections:
- net +3V3: now also JP2.1 (A)
- net +5V: now also JP1.1 (A)
- net at C2.1, C3.1, U1.2 (VO): now also JP2.2 (B)
- net at C1.1, U1.3 (VI): now also JP1.2 (B)
Changed lines of the file:
@@
 AR Path="/5C0BBB2B/5C0D4463" Ref="#PWR?"  Part="1"
 AR Path="/5C0BFA48/5C0D4463" Ref="#PWR?"  Part="1"
-AR Path="/5CF6369E/5C0D4463" Ref="#PWR0101"  Part="1"
-F 0 "#PWR0101" H 5750 2450 50  0001 C CNN
+AR Path="/5CF6369E/5C0D4463" Ref="#PWR011"  Part="1"
+F 0 "#PWR011" H 5750 2450 50  0001 C CNN
 F 1 "GND" H 5800 2500 50  0000 C CNN
 F 2 "" H 5750 2700 50  0001 C CNN
@@
 AR Path="/5C0BBB2B/5C0C105F" Ref="#PWR?"  Part="1"
 AR Path="/5C0BFA48/5C0C105F" Ref="#PWR?"  Part="1"
-AR Path="/5CF6369E/5C0C105F" Ref="#PWR0102"  Part="1"
-F 0 "#PWR0102" H 3750 2050 50  0001 C CNN
+AR Path="/5CF6369E/5C0C105F" Ref="#PWR09"  Part="1"
+F 0 "#PWR09" H 3750 2050 50  0001 C CNN
 F 1 "GND" H 3800 2100 50  0000 C CNN
 F 2 "" H 3750 2300 50  0001 C CNN
@@
 	3750 2250 3750 2300
 $Comp
-L power:+3V3 #PWR0103
+L power:+3V3 #PWR05
 U 1 1 5C0C1334
 P 3750 1750
-F 0 "#PWR0103" H 3750 1600 50  0001 C CNN
+F 0 "#PWR05" H 3750 1600 50  0001 C CNN
 F 1 "+3V3" H 3800 1950 50  0000 C CNN
 F 2 "" H 3750 1750 50  0001 C CNN
@@
 	0    -1   -1   0
 $EndComp
-$Comp
-L Device:Jumper_NO_Small JP1
-U 1 1 5C148323
-P 5050 1850
-F 0 "JP1" V 5000 1900 50  0000 L CNN
-F 1 "5V_EN" V 5050 1900 50  0000 L CNN
-F 2 "" H 5050 1850 50  0001 C CNN
-F 3 "~" H 5050 1850 50  0001 C CNN
-	1    5050 1850
-	0    1    1    0
-$EndComp
-Wire Wire Line
-	5050 1700 5050 1750
+Wire Wire Line
+	5050 1600 5050 1650
 Wire Wire Line
 	5050 1950 5050 2100
@@
 AR Path="/5C0BBB2B/5C14C0B1" Ref="#PWR?"  Part="1"
 AR Path="/5C0BFA48/5C14C0B1" Ref="#PWR?"  Part="1"
-AR Path="/5CF6369E/5C14C0B1" Ref="#PWR0104"  Part="1"
-F 0 "#PWR0104" H 5050 2450 50  0001 C CNN
+AR Path="/5CF6369E/5C14C0B1" Ref="#PWR010"  Part="1"
+F 0 "#PWR010" H 5050 2450 50  0001 C CNN
 F 1 "GND" H 5100 2500 50  0000 C CNN
 F 2 "" H 5050 2700 50  0001 C CNN
@@
 	5050 2400 5050 2700
 $Comp
-L power:+5V #PWR0105
+L power:+5V #PWR03
 U 1 1 5C153651
-P 5050 1700
-F 0 "#PWR0105" H 5050 1550 50  0001 C CNN
-F 1 "+5V" H 5100 1900 50  0000 C CNN
-F 2 "" H 5050 1700 50  0001 C CNN
-F 3 "" H 5050 1700 50  0001 C CNN
-	1    5050 1700
+P 5050 1600
+F 0 "#PWR03" H 5050 1450 50  0001 C CNN
+F 1 "+5V" H 5100 1800 50  0000 C CNN
+F 2 "" H 5050 1600 50  0001 C CNN
+F 3 "" H 5050 1600 50  0001 C CNN
+	1    5050 1600
 	1    0    0    -1
 $EndComp
@@
 F 0 "J1" H 892 1935 50  0000 C CNN
 F 1 "Vin" H 892 1844 50  0000 C CNN
-F 2 "" H 1000 1750 50  0001 C CNN
+F 2 "Connector_PinHeader_2.54mm:PinHeader_1x02_P2.54mm_Vertical" H 1000 1750 50  0001 C CNN
 F 3 "~" H 1000 1750 50  0001 C CNN
 	1    1000 1750
@@
 $EndComp
 $Comp
-L power:+5V #PWR0106
+L power:+5V #PWR01
 U 1 1 5CF6ACAF
 P 2150 1650
-F 0 "#PWR0106" H 2150 1500 50  0001 C CNN
+F 0 "#PWR01" H 2150 1500 50  0001 C CNN
 F 1 "+5V" H 2200 1850 50  0000 C CNN
 F 2 "" H 2150 1650 50  0001 C CNN
@@
 	1200 1750 1600 1750
 $Comp
-L power:GND #PWR0107
+L power:GND #PWR06
 U 1 1 5CF725A2
 P 1350 2050
-F 0 "#PWR0107" H 1350 1800 50  0001 C CNN
+F 0 "#PWR06" H 1350 1800 50  0001 C CNN
 F 1 "GND" H 1355 1877 50  0000 C CNN
 F 2 "" H 1350 2050 50  0001 C CNN
@@
 	1600 1750 1750 1750
 $Comp
-L power:GND #PWR0108
+L power:GND #PWR07
 U 1 1 5CF74691
 P 1600 2300
-F 0 "#PWR0108" H 1600 2050 50  0001 C CNN
+F 0 "#PWR07" H 1600 2050 50  0001 C CNN
 F 1 "GND" H 1605 2127 50  0000 C CNN
 F 2 "" H 1600 2300 50  0001 C CNN
@@
 	2150 1750 2150 1650
 Wire Wire Line
-	7250 1650 7250 1750
+	7250 1550 7250 1650
 Wire Wire Line
 	7150 2500 7250 2500
@@
 AR Path="/5C0BBB2B/5C14BD92" Ref="#PWR?"  Part="1"
 AR Path="/5C0BFA48/5C14BD92" Ref="#PWR?"  Part="1"
-AR Path="/5CF6369E/5C14BD92" Ref="#PWR0109"  Part="1"
-F 0 "#PWR0109" H 7150 2450 50  0001 C CNN
+AR Path="/5CF6369E/5C14BD92" Ref="#PWR012"  Part="1"
+F 0 "#PWR012" H 7150 2450 50  0001 C CNN
 F 1 "GND" H 7200 2500 50  0000 C CNN
 F 2 "" H 7150 2700 50  0001 C CNN
@@
 	7250 1950 7250 2100
 $Comp
-L Device:Jumper_NO_Small JP2
-U 1 1 5C148F3B
-P 7250 1850
-F 0 "JP2" V 7200 1900 50  0000 L CNN
-F 1 "3V3_EN" V 7250 1900 50  0000 L CNN
-F 2 "" H 7250 1850 50  0001 C CNN
-F 3 "~" H 7250 1850 50  0001 C CNN
-	1    7250 1850
-	0    1    1    0
-$EndComp
-$Comp
-L power:+3V3 #PWR0110
+L power:+3V3 #PWR02
 U 1 1 5C0C0902
-P 7250 1650
-F 0 "#PWR0110" H 7250 1500 50  0001 C CNN
-F 1 "+3V3" H 7300 1850 50  0000 C CNN
-F 2 "" H 7250 1650 50  0001 C CNN
-F 3 "" H 7250 1650 50  0001 C CNN
-	1    7250 1650
+P 7250 1550
+F 0 "#PWR02" H 7250 1400 50  0001 C CNN
+F 1 "+3V3" H 7300 1750 50  0000 C CNN
+F 2 "" H 7250 1550 50  0001 C CNN
+F 3 "" H 7250 1550 50  0001 C CNN
+	1    7250 1550
 	1    0    0    -1
 $EndComp
@@
 AR Path="/5C0BBB2B/5CFA8CD8" Ref="#PWR?"  Part="1"
 AR Path="/5C0BFA48/5CFA8CD8" Ref="#PWR?"  Part="1"
-AR Path="/5CF6369E/5CFA8CD8" Ref="#PWR0111"  Part="1"
-F 0 "#PWR0111" H 3000 2050 50  0001 C CNN
+AR Path="/5CF6369E/5CFA8CD8" Ref="#PWR08"  Part="1"
+F 0 "#PWR08" H 3000 2050 50  0001 C CNN
 F 1 "GND" H 3050 2100 50  0000 C CNN
 F 2 "" H 3000 2300 50  0001 C CNN
@@
 $EndComp
 $Comp
-L power:+5V #PWR0112
+L power:+5V #PWR04
 U 1 1 5CFAA1AE
 P 3000 1750
-F 0 "#PWR0112" H 3000 1600 50  0001 C CNN
+F 0 "#PWR04" H 3000 1600 50  0001 C CNN
 F 1 "+5V" H 3015 1923 50  0000 C CNN
 F 2 "" H 3000 1750 50  0001 C CNN
@@
 	1    0    0    -1
 $EndComp
+$Comp
+L my_solder_jumper:SolderJumper_2_Open_round JP1
+U 1 1 5CF87C61
+P 5050 1800
+F 0 "JP1" V 5004 1868 50  0000 L CNN
+F 1 "5V_EN" V 5095 1868 50  0000 L CNN
+F 2 "Jumper:SolderJumper-2_P1.3mm_Open_RoundedPad1.0x1.5mm" H 5050 1800 50  0001 C CNN
+F 3 "~" H 5050 1800 50  0001 C CNN
+	1    5050 1800
+	0    1    1    0
+$EndComp
+$Comp
+L my_solder_jumper:SolderJumper_2_Open_round JP2
+U 1 1 5CF8B62A
+P 7250 1800
+F 0 "JP2" V 7204 1868 50  0000 L CNN
+F 1 "3V3_EN" V 7295 1868 50  0000 L CNN
+F 2 "Jumper:SolderJumper-2_P1.3mm_Open_RoundedPad1.0x1.5mm" H 7250 1800 50  0001 C CNN
+F 3 "~" H 7250 1800 50  0001 C CNN
+	1    7250 1800
+	0    1    1    0
+$EndComp
 $EndSCHEMATC
