File: hardware/ESP12-breakout.sch (KiCad schematic (older format))
At the start: 0 parts

Commit message: update,
Other:
- note removed: "TODO: DELETE\n"
Changed lines of the file:
@@
 $Descr User 8500 5500
 encoding utf-8
-Sheet 1 9
+Sheet 1 8
 Title ""
 Date ""
@@
 F1 "one-wire.sch" 50
 F2 "DATA" I L 5850 2150 50
-$EndSheet
-$Sheet
-S -2250 750  900  500
-U 5CF63748
-F0 "uart" 50
-F1 "uart.sch" 50
 $EndSheet
 $Sheet
@@
 Wire Wire Line
 	2950 2050 3550 2050
-Text Notes -2100 1050 0    50   ~ 0
-TODO: DELETE\n
 Wire Wire Line
 	5200 2150 5850 2150

Commit message: update for 24C02,
Other:
- note added: "5 DRC error accepted"
Changed lines of the file:
@@
 $Descr User 8500 5500
 encoding utf-8
-Sheet 1 8
+Sheet 1 9
 Title ""
 Date ""
@@
 	5200 2150 5850 2150
 Wire Wire Line
-	2950 1250 3550 1250
+	2950 1250 3200 1250
 Wire Wire Line
-	2950 1350 3550 1350
+	2950 1350 3100 1350
 Wire Wire Line
 	2950 2850 3550 2850
@@
 Wire Wire Line
 	5200 1450 5850 1450
+Text Notes 3900 4100 0    100  ~ 0
+5 DRC error accepted
+$Sheet
+S 2050 550  900  400
+U 5CFAB75A
+F0 "24c02" 50
+F1 "24c02.sch" 50
+F2 "SCL" I R 2950 700 50
+F3 "SDA" I R 2950 800 50
+$EndSheet
+Wire Wire Line
+	2950 700  3200 700
+Wire Wire Line
+	3200 700  3200 1250
+Connection ~ 3200 1250
+Wire Wire Line
+	3200 1250 3550 1250
+Wire Wire Line
+	2950 800  3100 800
+Wire Wire Line
+	3100 800  3100 1350
+Connection ~ 3100 1350
+Wire Wire Line
+	3100 1350 3550 1350
 $EndSCHEMATC

Commit message: update for routing,
Parts:
- added H1, H2, H3, H4: MOUNT_M2.5, footprint-lib:MountingHole_2.7mm_M2.5,rpi_like, symbol taobao-mounting-hole:MOUNT_M2.5
Changed lines of the file:
@@
 Wire Wire Line
 	3100 1350 3550 1350
+$Comp
+L taobao-mounting-hole:MOUNT_M2.5 H1
+U 1 1 5CFC54DC
+P 3050 4100
+F 0 "H1" H 3150 4146 50  0000 L CNN
+F 1 "MOUNT_M2.5" H 3150 4055 50  0000 L CNN
+F 2 "footprint-lib:MountingHole_2.7mm_M2.5,rpi_like" H 3050 4100 50  0001 C CNN
+F 3 "~" H 3050 4100 50  0001 C CNN
+	1    3050 4100
+	1    0    0    -1
+$EndComp
+$Comp
+L taobao-mounting-hole:MOUNT_M2.5 H2
+U 1 1 5CFC5740
+P 3050 4300
+F 0 "H2" H 3150 4346 50  0000 L CNN
+F 1 "MOUNT_M2.5" H 3150 4255 50  0000 L CNN
+F 2 "footprint-lib:MountingHole_2.7mm_M2.5,rpi_like" H 3050 4300 50  0001 C CNN
+F 3 "~" H 3050 4300 50  0001 C CNN
+	1    3050 4300
+	1    0    0    -1
+$EndComp
+$Comp
+L taobao-mounting-hole:MOUNT_M2.5 H3
+U 1 1 5CFC5AD5
+P 3050 4500
+F 0 "H3" H 3150 4546 50  0000 L CNN
+F 1 "MOUNT_M2.5" H 3150 4455 50  0000 L CNN
+F 2 "footprint-lib:MountingHole_2.7mm_M2.5,rpi_like" H 3050 4500 50  0001 C CNN
+F 3 "~" H 3050 4500 50  0001 C CNN
+	1    3050 4500
+	1    0    0    -1
+$EndComp
+$Comp
+L taobao-mounting-hole:MOUNT_M2.5 H4
+U 1 1 5CFC5ADF
+P 3050 4700
+F 0 "H4" H 3150 4746 50  0000 L CNN
+F 1 "MOUNT_M2.5" H 3150 4655 50  0000 L CNN
+F 2 "footprint-lib:MountingHole_2.7mm_M2.5,rpi_like" H 3050 4700 50  0001 C CNN
+F 3 "~" H 3050 4700 50  0001 C CNN
+	1    3050 4700
+	1    0    0    -1
+$EndComp
 $EndSCHEMATC
