File: hardware/ESP12-breakout.kicad_pcb (KiCad board)
At the start: 2 copper layers, 90 x 90 mm, 43 parts, among them J1 Vin, J2 I2C, J3 ADC, J4 ONE_WIRE, J5 TTL_HEADER, J6 TF_HEADER, J7 IO, SW1 SW_RESET,2_leg,SMD, SW2 SW_RESET,2_leg,SMD, U1 AMS1117-3.3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

Commit message: update for 24C02,
Parts:
- added C8: C106,0805, Capacitor_SMD:C_0805_2012Metric_Pad1.15x1.40mm_HandSolder, F.Cu at (105.0, 93.5)
- added RN2: RN_472,0603, Resistor_SMD:R_Array_Concave_4x0603, F.Cu at (112.0, 100.0)
- added U5: 24C02_SOIC8, footprint-lib:24Cxx_SOIC8, F.Cu at (105.0, 98.0)
Connections:
- net /ESP-12E/SCL renamed /24c02/SCL
- net /ESP-12E/SDA renamed /24c02/SDA

Commit message: update for routing,
Parts:
- added H1: MOUNT_M2.5, footprint-lib:MountingHole_2.7mm_M2.5,rpi_like, F.Cu at (60.0, 140.0)
- added H2: MOUNT_M2.5, footprint-lib:MountingHole_2.7mm_M2.5,rpi_like, F.Cu at (140.0, 60.0)
- added H3: MOUNT_M2.5, footprint-lib:MountingHole_2.7mm_M2.5,rpi_like, F.Cu at (60.0, 60.0)
- added H4: MOUNT_M2.5, footprint-lib:MountingHole_2.7mm_M2.5,rpi_like, F.Cu at (140.0, 140.0)
- moved J2 28.0 mm to (131.5, 93.0)
- moved RN1 28.0 mm to (126.5, 97.0)
- moved J3 10.1 mm to (140.5, 94.0)
- moved R4 10.1 mm to (135.2, 99.0)
- moved R5 10.1 mm to (135.2, 94.6)
- moved J5 10.0 mm to (140.0, 75.0), turned to 180 degrees
- moved J7 9.96 mm to (125.5, 85.5)
- moved C4 8.63 mm to (122.5, 97.5)
- moved J4 8.63 mm to (117.1, 93.6)
- moved R6 8.63 mm to (120.5, 97.5)
- moved C7 6.58 mm to (69.0, 66.0)
Routing:
- net GND: track 0.00 -> 361.4 mm
- net +3V3: track 0.00 -> 242.6 mm, vias 0 -> 3
- net +5V: track 0.00 -> 97.7 mm
- net /ESP-12E/CS: track 0.00 -> 78.4 mm, vias 0 -> 2
- net /SDCARD/DO: track 0.00 -> 78.3 mm, vias 0 -> 1
- net /ESP-12E/DATA: track 0.00 -> 74.2 mm, vias 0 -> 1
- net /24c02/SCL: track 0.00 -> 73.8 mm
- net /SDCARD/CLK: track 0.00 -> 72.3 mm, vias 0 -> 3
- net /SDCARD/DI: track 0.00 -> 68.9 mm, vias 0 -> 1
- net /ESP-12E/ADC: track 0.00 -> 67.2 mm, vias 0 -> 2
- net /24c02/SDA: track 0.00 -> 61.8 mm, vias 0 -> 1
- net Net-(R10-Pad2): track 0.00 -> 42.7 mm, vias 0 -> 2
- net /SDCARD/CD: track 0.00 -> 32.2 mm, vias 0 -> 1
- net /ESP-12E/RESET: track 0.00 -> 32.1 mm
- net Net-(C2-Pad1): track 0.00 -> 26.8 mm
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Other:
- net class 300mA added: clearance 0.2, trace_width 0.4, via_dia 0.8, via_drill 0.4
- net class 800mA added: clearance 0.2, trace_width 0.5, via_dia 0.8, via_drill 0.4
- net class GND added: clearance 0.2, trace_width 0.25, via_dia 0.8, via_drill 0.4

Commit message: update for routing, DRC ok,
Routing:
- net /ESP-12E/ADC: track 67.2 -> 74.1 mm
- net Net-(R10-Pad2): track 42.7 -> 47.0 mm
- net /ESP-12E/DATA: track 74.2 -> 77.8 mm
- net GND: track 361.4 -> 364.4 mm
- net /24c02/SDA: track 61.8 -> 63.9 mm
- net /24c02/SCL: track 73.8 -> 75.6 mm
- net /ESP-12E/IO5: track 18.7 -> 19.8 mm, vias 0 -> 2

Commit message: update for routing, DRC ok,
Parts:
- moved J5 7.10 mm to (141.2, 68.0)
Routing:
- net /ESP-12E/CS: track 78.4 -> 104.9 mm
- net GND: track 364.4 -> 386.0 mm, vias 0 -> 5
- net /ESP-12E/ADC: track 74.1 -> 56.8 mm, vias 2 -> 4
- net /ESP-12E/RESET: track 32.1 -> 21.4 mm, vias 0 -> 2
- net /SDCARD/CLK: track 72.3 -> 82.7 mm
- net /SDCARD/DI: track 68.9 -> 79.2 mm, vias 1 -> 3
- net /24c02/SCL: track 75.6 -> 66.5 mm, vias 0 -> 1
- net Net-(R10-Pad2): track 47.0 -> 38.6 mm
- net Net-(D1-Pad1): track 15.1 -> 6.92 mm
- net /24c02/SDA: track 63.9 -> 71.5 mm
- net /ESP-12E/DATA: track 77.8 -> 84.5 mm
- net /ESP-12E/TXD: track 13.4 -> 7.23 mm
- net +3V3: track 242.6 -> 247.7 mm, vias 3 -> 4
- net /ESP-12E/IO5: track 19.8 -> 14.7 mm, vias 2 -> 1
- net +5V: track 97.7 -> 102.6 mm
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
Commit message: update for routing, DRC ok,
Routing:
- net GND: track 386.0 -> 389.1 mm, vias 5 -> 17
- net /ESP-12E/CS: track 104.9 -> 106.3 mm
- added copper zone on B.Cu, net GND
- added copper zone on F.Cu, net GND
Other:
- outline, holes or cut-outs redrawn
Changed lines of the file:
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@@
   (general
     (thickness 1.6)
-    (drawings 12)
-    (tracks 595)
+    (drawings 16)
+    (tracks 606)
     (zones 0)
     (modules 50)
@@
     )
   )
+  (gr_arc (start 60 140) (end 55 140) (angle -90) (layer Edge.Cuts) (width 0.05))
+  (gr_arc (start 140 140) (end 140 145) (angle -90) (layer Edge.Cuts) (width 0.05))
+  (gr_arc (start 140 60) (end 145 60) (angle -90) (layer Edge.Cuts) (width 0.05))
+  (gr_arc (start 60 60) (end 60 55) (angle -90) (layer Edge.Cuts) (width 0.05))
   (gr_line (start 56 142) (end 56 58) (layer Dwgs.User) (width 0.15))
   (gr_line (start 58 144) (end 56 142) (layer Dwgs.User) (width 0.15))
@@
   (gr_line (start 58 56) (end 142 56) (layer Dwgs.User) (width 0.15))
   (gr_line (start 56 58) (end 58 56) (layer Dwgs.User) (width 0.15))
-  (gr_line (start 145 55) (end 55 55) (layer Edge.Cuts) (width 0.05))
-  (gr_line (start 145 145) (end 145 55) (layer Edge.Cuts) (width 0.05))
-  (gr_line (start 55 145) (end 145 145) (layer Edge.Cuts) (width 0.05))
-  (gr_line (start 55 55) (end 55 145) (layer Edge.Cuts) (width 0.05))
+  (gr_line (start 140 55) (end 60 55) (layer Edge.Cuts) (width 0.05))
+  (gr_line (start 145 140) (end 145 60) (layer Edge.Cuts) (width 0.05))
+  (gr_line (start 60 145) (end 140 145) (layer Edge.Cuts) (width 0.05))
+  (gr_line (start 55 60) (end 55 140) (layer Edge.Cuts) (width 0.05))
   (via (at 120 66) (size 0.8) (drill 0.4) (layers F.Cu B.Cu) (net 29))
   (via (at 120 84.8) (size 0.8) (drill 0.4) (layers F.Cu B.Cu) (net 30))
@@
   (segment (start 103.975 86.4) (end 103.975 93.5) (width 0.25) (layer F.Cu) (net 1))
   (segment (start 100 86.4) (end 103.975 86.4) (width 0.25) (layer F.Cu) (net 1))
-  (segment (start 74.4832 64.0307) (end 74.4832 61.1753) (width 0.25) (layer F.Cu) (net 1))
-  (segment (start 70.8 66) (end 72.7693 64.0307) (width 0.25) (layer F.Cu) (net 1))
-  (segment (start 72.7693 64.0307) (end 74.4832 64.0307) (width 0.25) (layer F.Cu) (net 1))
   (segment (start 107.5625 97.365) (end 112.2 97.365) (width 0.25) (layer F.Cu) (net 1))
   (segment (start 112.2 97.365) (end 115.965 93.6) (width 0.25) (layer F.Cu) (net 1))
@@
   (segment (start 59.1553 70.92) (end 61.7396 68.3357) (width 0.25) (layer F.Cu) (net 1))
   (segment (start 61.7396 68.3357) (end 65.4857 68.3357) (width 0.25) (layer F.Cu) (net 1))
-  (segment (start 77.58 60) (end 76.4047 60) (width 0.25) (layer F.Cu) (net 1))
-  (segment (start 76.4047 60) (end 76.4047 60.3673) (width 0.25) (layer F.Cu) (net 1))
-  (segment (start 76.4047 60.3673) (end 75.5967 61.1753) (width 0.25) (layer F.Cu) (net 1))
-  (segment (start 75.5967 61.1753) (end 74.4832 61.1753) (width 0.25) (layer F.Cu) (net 1))
-  (segment (start 72.5 60) (end 73.6753 60) (width 0.25) (layer F.Cu) (net 1))
-  (segment (start 73.6753 60) (end 73.6753 60.3674) (width 0.25) (layer F.Cu) (net 1))
-  (segment (start 73.6753 60.3674) (end 74.4832 61.1753) (width 0.25) (layer F.Cu) (net 1))
-  (segment (start 74.4832 64.0307) (end 74.9057 64.0307) (width 0.25) (layer F.Cu) (net 1))
-  (segment (start 74.9057 64.0307) (end 80.875 70) (width 0.25) (layer F.Cu) (net 1))
   (segment (start 107.5 58.2) (end 107.419 58.1186) (width 0.25) (layer F.Cu) (net 1))
   (segment (start 107.419 58.1186) (end 71.2166 58.1186) (width 0.25) (layer F.Cu) (net 1))
@@
   (segment (start 139.4 94) (end 140.5 94) (width 0.25) (layer F.Cu) (net 1))
   (segment (start 138.2 92.8) (end 139.4 94) (width 0.25) (layer F.Cu) (net 1))
-  (segment (start 132.8 92.8) (end 138.2 92.8) (width 0.25) (layer F.Cu) (net 1))
+  (segment (start 132.8 92.8) (end 137.2 92.8) (width 0.25) (layer F.Cu) (net 1))
   (segment (start 133.823478 95.515) (end 132.854239 94.545761) (width 0.25) (layer F.Cu) (net 1))
   (segment (start 135.15 95.515) (end 133.823478 95.515) (width 0.25) (layer F.Cu) (net 1))
@@
   (segment (start 139.774976 83.025024) (end 141 81.8) (width 0.25) (layer B.Cu) (net 1))
   (segment (start 125.5 85.5) (end 125.5 84.4) (width 0.25) (layer B.Cu) (net 1))
+  (segment (start 80.875 70) (end 80.875 67.075) (width 0.25) (layer F.Cu) (net 1))
+  (segment (start 77.58 63.78) (end 77.58 60) (width 0.25) (layer F.Cu) (net 1))
+  (segment (start 80.875 67.075) (end 77.58 63.78) (width 0.25) (layer F.Cu) (net 1))
+  (segment (start 75.36 66) (end 77.58 63.78) (width 0.25) (layer F.Cu) (net 1))
+  (segment (start 70.8 66) (end 75.36 66) (width 0.25) (layer F.Cu) (net 1))
+  (segment (start 72.5 62.3) (end 72.5 60) (width 0.25) (layer F.Cu) (net 1))
+  (segment (start 70.8 66) (end 70.8 64) (width 0.25) (layer F.Cu) (net 1))
+  (segment (start 70.8 64) (end 72.5 62.3) (width 0.25) (layer F.Cu) (net 1))
+  (via (at 95 75) (size 0.8) (drill 0.4) (layers F.Cu B.Cu) (net 1))
+  (via (at 84 70) (size 0.8) (drill 0.4) (layers F.Cu B.Cu) (net 1))
+  (via (at 81 64) (size 0.8) (drill 0.4) (layers F.Cu B.Cu) (net 1))
+  (via (at 87 64) (size 0.8) (drill 0.4) (layers F.Cu B.Cu) (net 1))
+  (via (at 80 74) (size 0.8) (drill 0.4) (layers F.Cu B.Cu) (net 1))
+  (via (at 80 76) (size 0.8) (drill 0.4) (layers F.Cu B.Cu) (net 1))
+  (via (at 122 82) (size 0.8) (drill 0.4) (layers F.Cu B.Cu) (net 1))
+  (segment (start 137.2 92.8) (end 138.2 92.8) (width 0.25) (layer F.Cu) (net 1))
+  (via (at 137.2 92.8) (size 0.8) (drill 0.4) (layers F.Cu B.Cu) (net 1))
+  (via (at 84 63.9) (size 0.8) (drill 0.4) (layers F.Cu B.Cu) (net 1))
+  (via (at 71.8 75.8) (size 0.8) (drill 0.4) (layers F.Cu B.Cu) (net 1))
+  (via (at 124.2 99.4) (size 0.8) (drill 0.4) (layers F.Cu B.Cu) (net 1))
+  (via (at 127.1 100) (size 0.8) (drill 0.4) (layers F.Cu B.Cu) (net 1))
   (segment (start 65 94.65) (end 65 98.25) (width 0.25) (layer F.Cu) (net 2))
   (via (at 65 98.25) (size 0.8) (drill 0.4) (layers F.Cu B.Cu) (net 2))
@@
   (segment (start 87.74 60) (end 87.74 71.26) (width 0.25) (layer B.Cu) (net 20))
   (segment (start 87.74 71.26) (end 87.74 71.4927) (width 0.25) (layer B.Cu) (net 20))
-  (segment (start 137.8 80.4) (end 137.8 76.565685) (width 0.25) (layer B.Cu) (net 20))
-  (segment (start 120 86.6) (end 125.563498 81.036502) (width 0.25) (layer B.Cu) (net 20))
-  (segment (start 133.563498 81.036502) (end 134.451998 81.925002) (width 0.25) (layer B.Cu) (net 20))
-  (segment (start 134.451998 81.925002) (end 136.274998 81.925002) (width 0.25) (layer B.Cu) (net 20))
+  (via (at 137.8 76) (size 0.8) (drill 0.4) (layers F.Cu B.Cu) (net 20))
+  (segment (start 135.1 76) (end 137.8 76) (width 0.25) (layer F.Cu) (net 20))
   (segment (start 137.8 76.565685) (end 137.8 76) (width 0.25) (layer B.Cu) (net 20))
   (segment (start 136.274998 81.925002) (end 137.8 80.4) (width 0.25) (layer B.Cu) (net 20))
-  (segment (start 119.2 86.6) (end 120 86.6) (width 0.25) (layer B.Cu) (net 20))
-  (segment (start 118 85.4) (end 119.2 86.6) (width 0.25) (layer B.Cu) (net 20))
-  (segment (start 118 78.273004) (end 118 85.4) (width 0.25) (layer B.Cu) (net 20))
-  (segment (start 116.274998 76.548002) (end 118 78.273004) (width 0.25) (layer B.Cu) (net 20))
+  (segment (start 133.563498 81.036502) (end 134.451998 81.925002) (width 0.25) (layer B.Cu) (net 20))
+  (segment (start 125.563498 81.036502) (end 133.563498 81.036502) (width 0.25) (layer B.Cu) (net 20))
+  (segment (start 137.8 80.4) (end 137.8 76.565685) (width 0.25) (layer B.Cu) (net 20))
+  (segment (start 122.8 86.2) (end 122.8 83.8) (width 0.25) (layer B.Cu) (net 20))
+  (segment (start 122.4 86.6) (end 122.8 86.2) (width 0.25) (layer B.Cu) (net 20))
+  (segment (start 119.2 86.6) (end 122.4 86.6) (width 0.25) (layer B.Cu) (net 20))
   (segment (start 115.370154 71.26) (end 116.274998 72.164844) (width 0.25) (layer B.Cu) (net 20))
   (segment (start 116.274998 72.164844) (end 116.274998 76.548002) (width 0.25) (layer B.Cu) (net 20))
-  (via (at 137.8 76) (size 0.8) (drill 0.4) (layers F.Cu B.Cu) (net 20))
-  (segment (start 135.1 76) (end 137.8 76) (width 0.25) (layer F.Cu) (net 20))
   (segment (start 87.74 71.26) (end 115.370154 71.26) (width 0.25) (layer B.Cu) (net 20))
-  (segment (start 125.563498 81.036502) (end 133.563498 81.036502) (width 0.25) (layer B.Cu) (net 20))
+  (segment (start 116.274998 76.548002) (end 118 78.273004) (width 0.25) (layer B.Cu) (net 20))
+  (segment (start 134.451998 81.925002) (end 136.274998 81.925002) (width 0.25) (layer B.Cu) (net 20))
+  (segment (start 118 78.273004) (end 118 85.4) (width 0.25) (layer B.Cu) (net 20))
+  (segment (start 122.8 83.8) (end 125.563498 81.036502) (width 0.25) (layer B.Cu) (net 20))
+  (segment (start 118 85.4) (end 119.2 86.6) (width 0.25) (layer B.Cu) (net 20))
   (segment (start 74.5136 78.14) (end 74.4 78.0264) (width 0.25) (layer F.Cu) (net 21))
   (segment (start 76.85 78.14) (end 74.5136 78.14) (width 0.25) (layer F.Cu) (net 21))
@@
       )
     )
+  )
+  (zone (net 1) (net_name GND) (layer F.Cu) (hatch edge 0.508)
+    (connect_pads (clearance 0.508))
+    (min_thickness 0.254)
+    (fill yes (arc_segments 32) (thermal_gap 0.508) (thermal_bridge_width 0.508))
+    (polygon
+      (pts
+        (xy 50 50) (xy 50 150) (xy 150 150) (xy 150 50)
+      )
+    )
+  )
+  (zone (net 1) (net_name GND) (layer B.Cu) (hatch edge 0.508)
+    (connect_pads (clearance 0.508))
+    (min_thickness 0.254)
+    (fill yes (arc_segments 32) (thermal_gap 0.508) (thermal_bridge_width 0.508))
+    (polygon
+      (pts
+        (xy 50 50) (xy 50 150) (xy 150 150) (xy 150 50)
+      )
+    )
